File: fukc10X/fukc10X.kicad_pcb (KiCad board)
At the start: 2 copper layers, 427.1 x 117.5 mm, 274 parts, among them J1 SM04B-SRSS-TB, J2 Conn_01x02_Pin, J3 Conn_01x02_Pin, J4 Conn_01x02_Pin, J5 Conn_01x02_Pin, J6 Conn_01x02_Pin, J7 Conn_01x02_Pin, J8 Conn_01x02_Pin, U1 XC6206P332MR, U2 STM32F072CBT6

Commit message: updated LED Symbols + removed unnessecarry components for ESD and fusing
Parts:
- removed D1: PRTR5V0U2X, Package_TO_SOT_SMD:SOT-143
- removed F1: 500mA, Fuse:Fuse_1206_3216Metric
Connections:
- J1 pad 1: VBUS -> +5V
Routing:
- net +5V: track 580.6 -> 590.1 mm, vias 6 -> 8
- net VBUS: track 5.44 -> 0.00 mm
- net GND: track 95.8 -> 90.6 mm, vias 23 -> 21
- net COL9: track 275.4 -> 274.7 mm
- net COL8: track 283.7 -> 283.0 mm
- net COL7: track 336.1 -> 335.4 mm
- net D-: track 68.5 -> 67.9 mm
- net D+: track 68.5 -> 67.9 mm
