File: fukc10X/fukc10X.kicad_pcb (KiCad board)
At the start: 2 copper layers, 427.1 x 117.5 mm, 272 parts, among them J1 SM04B-SRSS-TB, J2 Conn_01x02_Pin, J3 Conn_01x02_Pin, J4 Conn_01x02_Pin, J5 Conn_01x02_Pin, J6 Conn_01x02_Pin, J7 Conn_01x02_Pin, J8 Conn_01x02_Pin, U1 XC6206P332MR, U2 STM32F072CBT6

Commit message: added back keys above numpad + updated step file/prod stuff
Parts:
- added D63: D_Small, Diode_SMD:D_SOD-123, B.Cu at (496.9, 104.3)
- added D78: D_Small, Diode_SMD:D_SOD-123, B.Cu at (477.8, 104.2)
- added MX126: MX_SW_solder, PCM_marbastlib-mx:SW_MX_1u, F.Cu at (493.7, 103.5)
- added MX127: MX_SW_solder, PCM_marbastlib-mx:SW_MX_1u, F.Cu at (474.7, 103.5)
- J2, J3, J4, J5, J6, J7, J8: value Conn_01x02_Pin -> LED_Conn01x02_Pin
- moved D116 300.6 mm to (201.3, 198.7)
- moved D117 300.6 mm to (195.7, 198.7)
- moved D119 300.6 mm to (206.8, 201.5)
- moved D120 300.6 mm to (201.3, 201.5)
- moved D121 300.6 mm to (195.7, 201.5)
- moved D66 300.6 mm to (206.8, 198.7)
- moved J6 6.23 mm to (455.6, 97.4)
- moved J7 6.23 mm to (455.6, 103.5)
- moved J8 6.23 mm to (455.6, 109.6)
Routing:
- net COL19: track 150.7 -> 174.8 mm
- net COL18: track 131.5 -> 155.5 mm
- net +5V: track 590.1 -> 612.2 mm, vias 8 -> 9
- net LedNum: track 108.7 -> 115.0 mm
- net LedCaps: track 513.4 -> 519.5 mm
- net LedScroll: track 112.2 -> 118.0 mm
- net Net-(D63-A): track 0.00 -> 4.50 mm
- net Net-(D78-A): track 0.00 -> 4.48 mm
- net ROW0: track 498.9 -> 495.0 mm
Other:
- board text removed: "<---- Minus"
