File: fukc10X/fukc10X.kicad_pcb (KiCad board)
At the start: 2 copper layers, 427.1 x 117.5 mm, 276 parts, among them J1 SM04B-SRSS-TB, J2 LED_Conn01x02_Pin, J3 LED_Conn01x02_Pin, J4 LED_Conn01x02_Pin, J5 LED_Conn01x02_Pin, J6 LED_Conn01x02_Pin, J7 LED_Conn01x02_Pin, J8 LED_Conn01x02_Pin, U1 XC6206P332MR, U2 STM32F072CBT6

Commit message: Soutfacing spacebar + zero Diode moved
Parts:
- moved D114 19.9 mm to (448.3, 204.3)
- turned S2 to 0 degrees
- turned S10 to 0 degrees
Routing:
- net Net-(D114-A): track 15.9 -> 22.3 mm
- net ROW5: track 479.3 -> 477.4 mm
- net ROW3: track 584.1 -> 582.5 mm
- net ROW4: track 451.9 -> 450.7 mm
Other:
- board size 427.1 x 117.5 mm -> 427.1 x 120.2 mm
