File: fukc10x_north/fukc10x_north.kicad_pcb (KiCad board)
At the start: 2 copper layers, 427.1 x 117.5 mm, 276 parts, among them J1 SM04B-SRSS-TB, J2 LED_Conn01x02_Pin, J3 LED_Conn01x02_Pin, J4 LED_Conn01x02_Pin, J5 LED_Conn01x02_Pin, J6 LED_Conn01x02_Pin, J7 LED_Conn01x02_Pin, J8 LED_Conn01x02_Pin, U1 XC6206P332MR, U2 STM32F072CBT6

Commit message: south version currently depreciated. Slight outline errors fixed on north version, aswell as traces adjusted/diodes moved to allow for shims when used with 1.2mm thickness. Indicator led were also ever so slightly off
Parts:
- moved D113 14.9 mm to (501.4, 201.1)
- moved D82 6.83 mm to (512.2, 171.9), turned to 0 degrees
- moved D115 5.15 mm to (483.0, 204.3)
Routing:
- net ROW5: track 477.4 -> 462.2 mm
- net Net-(D113-A): track 4.55 -> 14.3 mm
- net Net-(D82-A): track 4.55 -> 13.0 mm
- net ROW3: track 582.5 -> 575.7 mm
- net Net-(D115-A): track 4.55 -> 8.84 mm
- net COL8: track 283.0 -> 281.5 mm
- net COL9: track 274.7 -> 273.5 mm
- net COL2: track 398.6 -> 397.4 mm
- net COL0: track 432.7 -> 433.9 mm
- net COL1: track 416.4 -> 417.4 mm
- net COL10: track 265.7 -> 264.9 mm
- net COL11: track 250.7 -> 250.1 mm
- net +5V: vias 9 -> 10
Other:
- board text added: "Github repo for this PCB <--"
