File: fukc10x_north/fukc10x_north.kicad_pcb (KiCad board)
At the start: 2 copper layers, 427.1 x 117.5 mm, 270 parts, among them J1 SM04B-SRSS-TB, J2 LED_Conn01x02_Pin, J3 LED_Conn01x02_Pin, J4 LED_Conn01x02_Pin, J5 LED_Conn01x02_Pin, J6 LED_Conn01x02_Pin, J7 LED_Conn01x02_Pin, J8 LED_Conn01x02_Pin, U1 XC6206P332MR, U2 STM32F072CBT6

Commit message: fixed some shenanaigans
Parts:
- MX110: footprint acheron_MX_SolderMask:MX100 -> acheron_MX_SolderMask:MX200R
- MX77: footprint acheron_MX_SolderMask:MX250R -> acheron_MX_SolderMask:MX225R
- MX82: footprint acheron_MX_SolderMask:MX250 -> acheron_MX_SolderMask:MX225; moved to F.Cu
- moved MX115 0.79 mm to (105.6, 184.4)
- turned MX82 to 0 degrees
Connections:
- MX64 pad 1: COL0 -> Net-(D65-A)
- MX64 pad 2: Net-(D65-A) -> COL0
Routing:
- net Net-(D65-A): track 15.3 -> 12.3 mm
- net COL0: track 433.5 -> 431.1 mm
