File: fukc10x_north/matrix.kicad_sch (KiCad schematic)
At the start: 240 parts

Commit message: finishing touches (hopefully)
Parts:
- MX1: value MX_SW_solder -> Esc
- MX10: value MX_SW_solder -> F9
- MX100: value MX_SW_solder -> FN
- MX101: value MX_SW_solder -> Up
- MX102: value MX_SW_solder -> 1
- MX103: value MX_SW_solder -> 2
- MX104: value MX_SW_solder -> 3
- MX105: value MX_SW_solder -> Enter
- MX106, MX122: value MX_SW_solder -> Split Enter
- MX107, MX116: value MX_SW_solder -> Control
- MX108, MX113, MX114: value MX_SW_solder -> Super
- MX109: value MX_SW_solder -> Alt
- MX11: value MX_SW_solder -> F10
- MX110: value MX_SW_solder -> 6u Space
- MX111: value MX_SW_solder -> 7u Space
- MX112: value MX_SW_solder -> Alt Gr
- MX115: value MX_SW_solder -> Menu
- MX117: value MX_SW_solder -> Left
- MX118: value MX_SW_solder -> Down
- MX119: value MX_SW_solder -> Right
- MX12: value MX_SW_solder -> F11
- MX120: value MX_SW_solder -> Stabilized Zero
- MX121: value MX_SW_solder -> .del
- MX123: value MX_SW_solder -> 00
- MX124: value MX_SW_solder -> 0
- MX125: value alps capslock 1.5u -> Caps Alps
- MX126: value MX_SW_solder -> Alps Plus
- MX127: value MX_SW_solder -> Alps Enter
- MX13: value MX_SW_solder -> F12
- MX14: value MX_SW_solder -> PrtScr
- MX15: value MX_SW_solder -> ScrLck
- MX16: value MX_SW_solder -> Pause
- MX17: value MX_SW_solder -> M1
- MX18: value MX_SW_solder -> M2
- MX19: value MX_SW_solder -> M3
- MX2: value MX_SW_solder -> F1
- MX20: value MX_SW_solder -> ~`
- MX21: value MX_SW_solder -> 1!
- MX22: value MX_SW_solder -> 2@
- MX23: value MX_SW_solder -> 3#
- MX24: value MX_SW_solder -> 4$
- MX25: value MX_SW_solder -> 5%
- MX26: value MX_SW_solder -> 6^
- MX27: value MX_SW_solder -> 7&
- MX28: value MX_SW_solder -> 8*
- MX29: value MX_SW_solder -> 9(
- MX3: value MX_SW_solder -> F2
- MX30: value MX_SW_solder -> 0)
- MX31: value MX_SW_solder -> -_
- MX32: value MX_SW_solder -> =+
- MX33: value MX_SW_solder -> Split BS left
- MX34: value MX_SW_solder -> Backspace
- MX35: value MX_SW_solder -> Insert
- MX36: value MX_SW_solder -> Home
- MX37: value MX_SW_solder -> PgUp
- MX38: value MX_SW_solder -> Num Lock
- MX39: value MX_SW_solder -> Div
- MX4: value MX_SW_solder -> F3
- MX40: value MX_SW_solder -> Mult
- MX41: value MX_SW_solder -> Minus
- MX42: value MX_SW_solder -> Tab
- MX43: value MX_SW_solder -> Q
- MX44: value MX_SW_solder -> W
- MX45: value MX_SW_solder -> E
- MX46: value MX_SW_solder -> R
- MX47: value MX_SW_solder -> T
- MX48: value MX_SW_solder -> Y
- MX49: value MX_SW_solder -> U
- MX5: value MX_SW_solder -> F4
- MX50: value MX_SW_solder -> I
- MX51: value MX_SW_solder -> O
- MX52: value MX_SW_solder -> P
- MX53: value MX_SW_solder -> [{
- MX54: value MX_SW_solder -> ]}
- MX55: value MX_SW_solder -> \|
- MX56: value MX_SW_solder -> ISO Enter
- MX57: value MX_SW_solder -> delete
- MX58: value MX_SW_solder -> end
- MX59: value MX_SW_solder -> PgDn
- MX6: value MX_SW_solder -> F5
- MX60: value MX_SW_solder -> 7
- MX61: value MX_SW_solder -> 8
- MX62: value MX_SW_solder -> 9
- MX63: value MX_SW_solder -> Plus
- MX64, MX84: value MX_SW_solder -> Split Plus
- MX65: value MX_SW_solder -> Caps
- MX66: value MX_SW_solder -> CapsStep
- MX67: value MX_SW_solder -> A
- MX68: value MX_SW_solder -> S
- MX69: value MX_SW_solder -> D
- MX7: value MX_SW_solder -> F6
- MX70: value MX_SW_solder -> F
- MX71: value MX_SW_solder -> G
- MX72: value MX_SW_solder -> H
- MX73: value MX_SW_solder -> J
- MX74: value MX_SW_solder -> K
- MX75: value MX_SW_solder -> L
- MX76: value MX_SW_solder -> ;:
- MX77: value MX_SW_solder -> '"
- MX78: value MX_SW_solder -> NUHS
- MX79: value MX_SW_solder -> ANSI Enter
- MX8: value MX_SW_solder -> F7
- MX80: value MX_SW_solder -> Split Backspace right
- MX81: value MX_SW_solder -> 4
- MX82: value MX_SW_solder -> 5
- MX83: value MX_SW_solder -> 6
- MX85: value MX_SW_solder -> ANSI Shift
- MX86: value MX_SW_solder -> ISO Shift
- MX87: value MX_SW_solder -> NUBS
- MX88: value MX_SW_solder -> Z
- MX89: value MX_SW_solder -> X
- MX9: value MX_SW_solder -> F8
- MX90: value MX_SW_solder -> C
- MX91: value MX_SW_solder -> V
- MX92: value MX_SW_solder -> B
- MX93: value MX_SW_solder -> N
- MX94: value MX_SW_solder -> M
- MX95: value MX_SW_solder -> ,<
- MX96: value MX_SW_solder -> .>
- MX97: value MX_SW_solder -> /?
- MX98: value MX_SW_solder -> Split shift
- MX99: value MX_SW_solder -> Right shift
Other:
- moved on the sheet: D99, MX125, MX66, MX85, MX98, MX99

Commit message: idk changed a lot
Connections:
- net COL17: now also MX120.1, MX123.1; no longer MX120.2, MX123.2
- net COL20: now also MX122.1; no longer MX122.2
- net at D118.2 (A): now also MX122.2; no longer MX122.1
- new net: D119.2 (A), MX120.2, MX123.2
Other:
- moved on the sheet: MX120, MX122, MX123
Changed lines of the file:
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@@
 	)
 	(junction
+		(at 299.72 153.67)
+		(diameter 0)
+		(color 0 0 0 0)
+	)
+	(junction
 		(at 181.61 82.55)
 		(diameter 0)
@@
 	)
 	(junction
-		(at 299.72 153.67)
-		(diameter 0)
-		(color 0 0 0 0)
-	)
-	(junction
 		(at 25.4 95.25)
 		(diameter 0)
@@
 	)
 	(junction
-		(at 294.64 125.73)
-		(diameter 0)
-		(color 0 0 0 0)
-	)
-	(junction
 		(at 190.5 72.39)
 		(diameter 0)
@@
 	)
 	(junction
+		(at 294.64 125.73)
+		(diameter 0)
+		(color 0 0 0 0)
+	)
+	(junction
 		(at 176.53 72.39)
 		(diameter 0)
@@
 	(wire
 		(pts
-			(xy 294.64 125.73) (xy 294.64 148.59)
-		)
-		(stroke
-			(width 0)
-			(type default)
-		)
-	)
-	(wire
-		(pts
 			(xy 336.55 33.02) (xy 336.55 54.61)
 		)
@@
 	(wire
 		(pts
+			(xy 294.64 125.73) (xy 294.64 148.59)
+		)
+		(stroke
+			(width 0)
+			(type default)
+		)
+	)
+	(wire
+		(pts
 			(xy 350.52 113.03) (xy 360.68 113.03)
 		)
@@
 	(wire
 		(pts
+			(xy 299.72 130.81) (xy 299.72 153.67)
+		)
+		(stroke
+			(width 0)
+			(type default)
+		)
+	)
+	(wire
+		(pts
 			(xy 204.47 54.61) (xy 204.47 72.39)
 		)
@@
 	(wire
 		(pts
-			(xy 299.72 130.81) (xy 299.72 153.67)
-		)
-		(stroke
-			(width 0)
-			(type default)
-		)
-	)
-	(wire
-		(pts
 			(xy 120.65 33.02) (xy 120.65 54.61)
 		)
@@
 	(symbol
 		(lib_id "PCM_marbastlib-mx:MX_SW_solder")
-		(at 339.09 128.27 180)
+		(at 339.09 128.27 0)
 		(unit 1)
 		(body_style 1)
@@
 	(symbol
 		(lib_id "PCM_marbastlib-mx:MX_SW_solder")
-		(at 297.18 151.13 180)
+		(at 297.18 151.13 0)
 		(unit 1)
 		(body_style 1)
@@
 	(symbol
 		(lib_id "PCM_marbastlib-mx:MX_SW_solder")
-		(at 297.18 128.27 180)
+		(at 297.18 128.27 0)
 		(unit 1)
 		(body_style 1)
